File: project/controller.sch (KiCad schematic (older format))
At the start: 90 parts, among them IC1 ATMEGA1284-P, J1 USB_2_UPDATE, K1 X_MIN, K2 X_MAX, K3 Y_MIN, K4 Y_MAX, K5 Z_MIN, K6 Z_MAX, K7 RELAY_2RT, K8 RELAY_2RT, P1 ISP, P10 CONN_4, P11 CONN_4, P12 CONN_8, P13 CONN_8, P14 CONN_8, P15 CONN_8, P16 CONN_8, P17 CONN_8, P18 CONN_3X2, P19 CONN_3X2, P2 M1_IN, P20 CONN_3X2, P21 M_PWR, P22 PIN_HEADER, P23 I2C, P24 Z_PROBE, P25 12Volts, P26 5Volts, P27 R1_IN, P28 R2_IN, P29 R1_OUT, P3 M1_OUT, P30 R2_OUT, P31 MOUNT, P32 MOUNT, P33 MOUNT, P34 MOUNT, P4 M2_IN, P5 M2_OUT, P6 X_AXIS, P7 Y_AXIS, P8 Z_AXIS, P9 CONN_4, Q1 MOSFET_N, Q2 MOSFET_N, Q3 PN2222A, Q4 PN2222A, U1 7805, U2 FT230X, X1 CRYSTAL

Commit message: Latest files
Parts:
- removed C10: 47pF, symbol CSMALL
- removed R14: 4k7, symbol R
- removed R15: 10k, symbol R
- removed U2: FT230X, MODULE, symbol FT230X
- added D3, D4: LED, symbol LED
- added U2: FT232RL, symbol FT232RL
- C9: value 47pF -> 100nF
- R12, R13: value 27R -> 220
Connections:
- wire segments 354 -> 353

Commit message: Latest with GND pour
Parts:
- removed K1: X_MIN, symbol CONN_3
- removed K2: X_MAX, symbol CONN_3
- removed K3: Y_MIN, symbol CONN_3
- removed K4: Y_MAX, symbol CONN_3
- removed K5: Z_MIN, symbol CONN_3
- removed K6: Z_MAX, symbol CONN_3
- added K1: X_MIN, symbol CONN_2
- added K2: X_MAX, symbol CONN_2
- added K3: Y_MIN, symbol CONN_2
- added K4: Y_MAX, symbol CONN_2
- added K5: Z_MIN, symbol CONN_2
- added K6: Z_MAX, symbol CONN_2
Connections:
- wire segments 353 -> 346
